File: multiple/multiple.kicad_sch (KiCad schematic)
At the start: 25 parts, among them J1 Power Connector, J2 Input 1, J3 Input 2, J4 Output 5, J5 Output 6, J6 Output 4, J7 Output 1, J8 Output 2, J9 Output 3, U1 TL074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

Commit message: Added BOM for REV1
Parts:
- U1, U2: Manufacturer (none) -> VARIOUS; Manufacturer Part No. (none) -> TL074CN; Supplier (none) -> Tayda; Supplier Part No. (none) -> A-1138
Changed lines of the file:
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@@
+      (effects (font (size 1.27 1.27)) hide)
+    )
+    (property "Manufacturer" "VARIOUS" (id 4) (at 128.27 125.73 0)
+      (effects (font (size 1.27 1.27)) hide)
+    )
+    (property "Manufacturer Part No." "TL074CN" (id 5) (at 128.27 125.73 0)
+      (effects (font (size 1.27 1.27)) hide)
+    )
+    (property "Supplier" "Tayda" (id 6) (at 128.27 125.73 0)
+      (effects (font (size 1.27 1.27)) hide)
+    )
+    (property "Supplier Part No." "A-1138" (id 7) (at 128.27 125.73 0)
       (effects (font (size 1.27 1.27)) hide)
     )
@@
       (effects (font (size 1.27 1.27)) hide)
     )
+    (property "Manufacturer" "VARIOUS" (id 4) (at 130.81 167.64 0)
+      (effects (font (size 1.27 1.27)) hide)
+    )
+    (property "Manufacturer Part No." "TL074CN" (id 5) (at 130.81 167.64 0)
+      (effects (font (size 1.27 1.27)) hide)
+    )
+    (property "Supplier" "Tayda" (id 6) (at 130.81 167.64 0)
+      (effects (font (size 1.27 1.27)) hide)
+    )
+    (property "Supplier Part No." "A-1138" (id 7) (at 130.81 167.64 0)
+      (effects (font (size 1.27 1.27)) hide)
+    )
     (pin "1")
     (pin "2")
@@
       (effects (font (size 1.27 1.27)) hide)
     )
+    (property "Manufacturer" "VARIOUS" (id 4) (at 214.63 63.5 0)
+      (effects (font (size 1.27 1.27)) hide)
+    )
+    (property "Manufacturer Part No." "TL074CN" (id 5) (at 214.63 63.5 0)
+      (effects (font (size 1.27 1.27)) hide)
+    )
+    (property "Supplier" "Tayda" (id 6) (at 214.63 63.5 0)
+      (effects (font (size 1.27 1.27)) hide)
+    )
+    (property "Supplier Part No." "A-1138" (id 7) (at 214.63 63.5 0)
+      (effects (font (size 1.27 1.27)) hide)
+    )
     (pin "1")
     (pin "2")
@@
       (effects (font (size 1.27 1.27)) hide)
     )
+    (property "Manufacturer" "VARIOUS" (id 4) (at 214.63 95.25 0)
+      (effects (font (size 1.27 1.27)) hide)
+    )
+    (property "Manufacturer Part No." "TL074CN" (id 5) (at 214.63 95.25 0)
+      (effects (font (size 1.27 1.27)) hide)
+    )
+    (property "Supplier" "Tayda" (id 6) (at 214.63 95.25 0)
+      (effects (font (size 1.27 1.27)) hide)
+    )
+    (property "Supplier Part No." "A-1138" (id 7) (at 214.63 95.25 0)
+      (effects (font (size 1.27 1.27)) hide)
+    )
     (pin "1")
     (pin "2")
@@
       (effects (font (size 1.27 1.27)) hide)
     )
+    (property "Manufacturer" "VARIOUS" (id 4) (at 128.27 35.56 0)
+      (effects (font (size 1.27 1.27)) hide)
+    )
+    (property "Manufacturer Part No." "TL074CN" (id 5) (at 128.27 35.56 0)
+      (effects (font (size 1.27 1.27)) hide)
+    )
+    (property "Supplier" "Tayda" (id 6) (at 128.27 35.56 0)
+      (effects (font (size 1.27 1.27)) hide)
+    )
+    (property "Supplier Part No." "A-1138" (id 7) (at 128.27 35.56 0)
+      (effects (font (size 1.27 1.27)) hide)
+    )
     (pin "1")
     (pin "2")
@@
       (effects (font (size 1.27 1.27)) hide)
     )
+    (property "Manufacturer" "VARIOUS" (id 4) (at 128.27 95.25 0)
+      (effects (font (size 1.27 1.27)) hide)
+    )
+    (property "Manufacturer Part No." "TL074CN" (id 5) (at 128.27 95.25 0)
+      (effects (font (size 1.27 1.27)) hide)
+    )
+    (property "Supplier" "Tayda" (id 6) (at 128.27 95.25 0)
+      (effects (font (size 1.27 1.27)) hide)
+    )
+    (property "Supplier Part No." "A-1138" (id 7) (at 128.27 95.25 0)
+      (effects (font (size 1.27 1.27)) hide)
+    )
     (pin "1")
     (pin "2")
@@
       (effects (font (size 1.27 1.27)) hide)
     )
+    (property "Manufacturer" "VARIOUS" (id 4) (at 128.27 68.58 0)
+      (effects (font (size 1.27 1.27)) hide)
+    )
+    (property "Manufacturer Part No." "TL074CN" (id 5) (at 128.27 68.58 0)
+      (effects (font (size 1.27 1.27)) hide)
+    )
+    (property "Supplier" "Tayda" (id 6) (at 128.27 68.58 0)
+      (effects (font (size 1.27 1.27)) hide)
+    )
+    (property "Supplier Part No." "A-1138" (id 7) (at 128.27 68.58 0)
+      (effects (font (size 1.27 1.27)) hide)
+    )
     (pin "1")
     (pin "2")
@@
       (effects (font (size 1.27 1.27)) hide)
     )
+    (property "Manufacturer" "VARIOUS" (id 4) (at 214.63 34.29 0)
+      (effects (font (size 1.27 1.27)) hide)
+    )
+    (property "Manufacturer Part No." "TL074CN" (id 5) (at 214.63 34.29 0)
+      (effects (font (size 1.27 1.27)) hide)
+    )
+    (property "Supplier" "Tayda" (id 6) (at 214.63 34.29 0)
+      (effects (font (size 1.27 1.27)) hide)
+    )
+    (property "Supplier Part No." "A-1138" (id 7) (at 214.63 34.29 0)
+      (effects (font (size 1.27 1.27)) hide)
+    )
     (pin "1")
     (pin "2")
@@
       (effects (font (size 1.27 1.27)) hide)
     )
+    (property "Manufacturer" "VARIOUS" (id 4) (at 214.63 125.73 0)
+      (effects (font (size 1.27 1.27)) hide)
+    )
+    (property "Manufacturer Part No." "TL074CN" (id 5) (at 214.63 125.73 0)
+      (effects (font (size 1.27 1.27)) hide)
+    )
+    (property "Supplier" "Tayda" (id 6) (at 214.63 125.73 0)
+      (effects (font (size 1.27 1.27)) hide)
+    )
+    (property "Supplier Part No." "A-1138" (id 7) (at 214.63 125.73 0)
+      (effects (font (size 1.27 1.27)) hide)
+    )
     (pin "1")
     (pin "2")
@@
       (effects (font (size 1.27 1.27)) hide)
     )
+    (property "Manufacturer" "VARIOUS" (id 4) (at 152.4 167.64 0)
+      (effects (font (size 1.27 1.27)) hide)
+    )
+    (property "Manufacturer Part No." "TL074CN" (id 5) (at 152.4 167.64 0)
+      (effects (font (size 1.27 1.27)) hide)
+    )
+    (property "Supplier" "Tayda" (id 6) (at 152.4 167.64 0)
+      (effects (font (size 1.27 1.27)) hide)
+    )
+    (property "Supplier Part No." "A-1138" (id 7) (at 152.4 167.64 0)
+      (effects (font (size 1.27 1.27)) hide)
+    )
